File: Hardware/Auxiliary_Power_Supply.kicad_sch (KiCad schematic)
At the start: 26 parts, among them U2 RT9013-33GB, U9 LV14340DDAR

Commit message: feat: update footprint power supply
Parts:
- C10, C11, C13, C16, C17, C18, C19, C20, C27, C6, C8, C9: footprint (none) -> Capacitor_SMD:C_0805_2012Metric; Link to Buy (none) -> https://linhkien.cxtvn.com/1976-tu-khong-phan-cuc-0805.html
- C12: footprint (none) -> Capacitor_SMD:CP_Elec_5x5.4; Link to Buy (none) -> https://linhkien.cxtvn.com/9282-tu-nhom-100uf-10v-50x54mm.h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
- C7: value 100nF -> 100nF 50V; footprint (none) -> Capacitor_SMD:C_0805_2012Metric; Link to Buy (none) -> https://linhkien.cxtvn.com/1976-tu-khong-phan-cuc-0805.html
- D14: Link to Buy (none) -> https://linhkienchatluong.vn/urlled-dan-0603-smd/led-dan-06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
- D3, D8: LCSC Part (none) -> C2837271; Link to Buy (none) -> https://linhkien.cxtvn.com/1128-diode-ss34-sma-3a-40v-do-21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
- D4: value SMAJ36A -> SMAJ36CA; LCSC Part (none) -> C113967; Link to Buy (none) -> https://linhkienthuduc.com/san-pham/smaj36ca-tvs-diodes-400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
- F3: LCSC Part (none) -> C66453; Link to Buy (none) -> https://linhkienthuduc.com/san-pham/nsmd100-cau-chi-tu-phuc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; MPN (none) -> nSMD100
- L2: footprint (none) -> Inductor_SMD:L_SXN_SMDRI73; Link to Buy (none) -> https://linhkien.cxtvn.com/9904-cuon-cam-0630-cac-gia-tri.h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
- R10: footprint (none) -> Resistor_SMD:R_0603_1608Metric; Link to Buy (none) -> https://linhkienthuduc.com/san-pham/dien-tro-49-9-ohm-0603-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; MPN (none) -> 49R9 0603 1%
- R11: footprint (none) -> Resistor_SMD:R_0603_1608Metric; Link to Buy (none) -> https://linhkien.cxtvn.com/2304-dien-tro-68k-0603-1-100c.ht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
- R37: Link to Buy (none) -> https://linhkien.cxtvn.com/7112-dien-tro-0402-1-thong-so-tu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
- R48: footprint (none) -> Resistor_SMD:R_0603_1608Metric; Link to Buy (none) -> https://linhkienthuduc.com/san-pham/dien-tro-12k-ohm-0603-1/
- U2: LCSC Part (none) -> C47773; Link to Buy (none) -> https://linhkienthuduc.com/san-pham/rt9013-33gb-ic-nguon-ld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; MANUFACTURER (none) -> Richtek; MPN (none) -> RT9013-33GB
- U9: footprint SOIC8_DDA_TEX -> LV14340DDAR:SOIC8_DDA_TEX; LCSC Part (none) -> C882854; Link to Buy (none) -> https://banlinhkiendientu.vn/lv14340ddar-14340-ic-nguon-sop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; MANUFACTURER (none) -> Texas Instruments; MPN (none) -> LV14340DDAR

Commit message: feat: update schematic with new components for communication interfaces and export BOM list
Parts:
- C10: value 1u -> 1uF
- C11, C9: value 100n -> 100nF
- C12: value 100u -> 100uF
- C7: value 100nF 50V -> 100nF
- C8: value 10u -> 10uF
- D14: value GREEN -> LED_G
- F3: value Fuse 1A -> Fuse
- R10: value 49.9 -> 49.9R
- R11: value 68k -> 68kR
- R37: value 4.7k -> 4.7kR; footprint Resistor_SMD:R_0402_1005Metric_Pad0.72x0.64mm_HandSolder -> Resistor_SMD:R_0805_2012Metric; Link to Buy https://linhkien.cxtvn.com/7112-dien-tro-0402-1-thong-so-tu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 -> https://linhkien.cxtvn.com/6337-dien-tro-0805-1-thong-so-tu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
- R48: value 12k -> 12kR; footprint Resistor_SMD:R_0603_1608Metric -> Resistor_SMD:R_0805_2012Metric; Link to Buy https://linhkienthuduc.com/san-pham/dien-tro-12k-ohm-0603-1/ -> https://linhkien.cxtvn.com/4177-dien-tro-0805-1-thong-so-tu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
- U2: Link to Buy https://linhkienthuduc.com/san-pham/rt9013-33gb-ic-nguon-ld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 -> https://linhkienthuduc.com/san-pham/rt9013-33gb-jsm/; MANUFACTURER Richtek -> (none); Manufacturer (none) -> Richtek
- U9: MANUFACTURER Texas Instruments -> (none); Manufacturer (none) -> Texas Instruments
Changed lines of the file:
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@@
 			)
 		)
-		(property "Value" "68k"
+		(property "Value" "68kR"
 			(at 207.01 55.8799 0)
 			(show_name no)
@@
 			)
 		)
-		(property "Value" "GREEN"
+		(property "Value" "LED_G"
 			(at 254 67.2464 90)
 			(show_name no)
@@
 			)
 		)
-		(property "Value" "12k"
+		(property "Value" "12kR"
 			(at 207.01 73.6599 0)
 			(show_name no)
@@
 			)
 		)
-		(property "Footprint" "Resistor_SMD:R_0603_1608Metric"
+		(property "Footprint" "Resistor_SMD:R_0805_2012Metric"
 			(at 204.47 72.39 0)
 			(hide yes)
@@
 			)
 		)
-		(property "Link to Buy" "https://linhkienthuduc.com/san-pham/dien-tro-12k-ohm-0603-1/"
+		(property "Link to Buy" "https://linhkien.cxtvn.com/4177-dien-tro-0805-1-thong-so-tu-1k-den-91k.html"
 			(at 0 0 0)
 			(hide yes)
@@
 			)
 		)
-		(property "Value" "100n"
+		(property "Value" "100nF"
 			(at 60.96 127.0062 0)
 			(show_name no)
@@
 			)
 		)
-		(property "Value" "4.7k"
+		(property "Value" "4.7kR"
 			(at 254 55.8799 0)
 			(show_name no)
@@
 			)
 		)
-		(property "Footprint" "Resistor_SMD:R_0402_1005Metric_Pad0.72x0.64mm_HandSolder"
+		(property "Footprint" "Resistor_SMD:R_0805_2012Metric"
 			(at 251.46 54.61 0)
 			(hide yes)
@@
 			)
 		)
-		(property "Link to Buy" "https://linhkien.cxtvn.com/7112-dien-tro-0402-1-thong-so-tu-1k-den-91k.html"
+		(property "Link to Buy" "https://linhkien.cxtvn.com/6337-dien-tro-0805-1-thong-so-tu-1k-den-91k.html"
 			(at 0 0 0)
 			(hide yes)
@@
 			)
 		)
-		(property "Value" "10u"
+		(property "Value" "10uF"
 			(at 49.53 127.0062 0)
 			(show_name no)
@@
 			)
 		)
-		(property "Value" "Fuse 1A"
+		(property "Value" "Fuse"
 			(at 69.85 54.61 90)
 			(show_name no)
@@
 			)
 		)
-		(property "Datasheet" ""
+		(property "Datasheet" "https://www.lcsc.com/datasheet/C66453.pdf"
 			(at 69.85 58.42 0)
 			(hide yes)
@@
 			)
 		)
-		(property "Description" "Resettable fuse, polymeric positive temperature coefficient"
+		(property "Description" "Fuse 1A"
 			(at 69.85 58.42 0)
 			(hide yes)
@@
 			)
 		)
-		(property "Datasheet" "https://www.diodes.com/assets/Datasheets/AP2112.pdf"
+		(property "Datasheet" "https://www.lcsc.com/datasheet/C7434207.pdf"
 			(at 80.01 116.84 0)
 			(hide yes)
@@
 			)
 		)
-		(property "Link to Buy" "https://linhkienthuduc.com/san-pham/rt9013-33gb-ic-nguon-ldo-3-3v-500ma/"
+		(property "Link to Buy" "https://linhkienthuduc.com/san-pham/rt9013-33gb-jsm/"
 			(at 0 0 0)
 			(hide yes)
@@
 			)
 		)
-		(property "MANUFACTURER" "Richtek"
+		(property "Manufacturer" "Richtek"
 			(at 0 0 0)
 			(hide yes)
@@
 			)
 		)
-		(property "Value" "49.9"
+		(property "Value" "49.9R"
 			(at 116.84 71.1199 0)
 			(show_name no)
@@
 			)
 		)
-		(property "Value" "100nF 50V"
+		(property "Value" "100nF"
 			(at 118.1163 38.1 90)
 			(show_name no)
@@
 			)
 		)
-		(property "Value" "100u"
+		(property "Value" "100uF"
 			(at 128.27 127.3809 0)
 			(show_name no)
@@
 			)
 		)
-		(property "MANUFACTURER" "Texas Instruments"
+		(property "Manufacturer" "Texas Instruments"
 			(at 0 0 0)
 			(hide yes)
@@
 			)
 		)
-		(property "Value" "1u"
+		(property "Value" "1uF"
 			(at 100.33 127.0062 0)
 			(show_name no)
@@
 			)
 		)
-		(property "Value" "100n"
+		(property "Value" "100nF"
 			(at 111.76 127.0062 0)
 			(show_name no)
