File: Hardware/Communication_Interfaces.kicad_sch (KiCad schematic)
At the start: 59 parts, among them Q1 BCX56-16, Q11 MMBT3904, Q12 MMBT3904, Q6 BCX56-16, Q7 BCX56-16, U1 LTV-357T, U10 LTV-357T, U12 MCP2542FDxMF, U3 MAX3485, U6 LTV-357T

Commit message: feat: update schematic with new components for communication interfaces and export BOM list
Parts:
- removed D17, D18: D_TVS, symbol Device:D_TVS
- removed Q1, Q6, Q7: BCX56-16, Package_TO_SOT_SMD:SOT-23, symbol Transistor_BJT:BC817
- removed Q11, Q12: MMBT3904, Package_TO_SOT_SMD:SOT-23, symbol Transistor_BJT:MMBT3904
- removed U12: MCP2542FDxMF, Package_DFN_QFN:DFN-8-1EP_3x3mm_P0.65mm_EP1.55x2.4mm, symbol Interface_CAN_LIN:MCP2542FDxMF
- added D10, D11, D16, D18, D24: BZT52C12, Diode_SMD:D_SOD-123, symbol Diode:1N914
- added D9: SM712, Package_TO_SOT_SMD:SOT-23, symbol Diode:SM712_SOT23
- added Q1, Q11, Q12, Q6, Q7: SI2308BDS, Package_TO_SOT_SMD:SOT-23, symbol Transistor_FET:2N7002K
- added U12: TJA1051T-3, Package_SO:SOIC-8_3.9x4.9mm_P1.27mm, symbol Interface_CAN_LIN:TJA1051T-3
- C32, C37: value 47pF -> 33pF; footprint (none) -> Capacitor_SMD:C_0805_2012Metric; Link to Buy (none) -> https://linhkien.cxtvn.com/1976-tu-khong-phan-cuc-0805.html
- C33, C34, C35, C36, C38, C39, C40: footprint (none) -> Capacitor_SMD:C_0805_2012Metric; Link to Buy (none) -> https://linhkien.cxtvn.com/1976-tu-khong-phan-cuc-0805.html
- C4: value 0.1uF -> 100nF; footprint (none) -> Capacitor_SMD:C_0805_2012Metric; Link to Buy (none) -> https://linhkien.cxtvn.com/1976-tu-khong-phan-cuc-0805.html
- D1, D5, D6: value FR107 -> RS1M; footprint Diode_THT:D_DO-35_SOD27_P7.62mm_Horizontal -> Diode_SMD:D_SOD-123; Link to Buy (none) -> https://linhkien.cxtvn.com/9278-rs1m-fr107-f7-diode-xung-1a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; MPN (none) -> RS1M
- D19, D23: value ESD -> PESD5Z3.3; footprint Diode_SMD:D_SOD-923 -> Diode_SMD:D_SOD-323; LCSC Part (none) -> C96512; Link to Buy (none) -> https://linhkienthuduc.com/san-pham/pesd5z3-3/; MPN (none) -> PESD5Z3.3; Manufacturer (none) -> Nexperia
- D20, D21, D22: Link to Buy (none) -> https://linhkienchatluong.vn/urlled-dan-0603-smd/led-dan-06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
- D25, D26: value 1N914 -> 1N4148W; footprint Diode_THT:D_DO-35_SOD27_P7.62mm_Horizontal -> Diode_SMD:D_SOD-123; Link to Buy (none) -> https://linhkien.cxtvn.com/7017-1n4148w-7-f-diode-gen-purp-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; MPN (none) -> 1N4148
- R12, R38: value 10k -> 4.7kR; footprint (none) -> Resistor_SMD:R_0805_2012Metric; Link to Buy (none) -> https://linhkien.cxtvn.com/6337-dien-tro-0805-1-thong-so-tu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
- R13, R39: value 100k -> 150kR; footprint (none) -> Resistor_SMD:R_0805_2012Metric; Link to Buy (none) -> https://linhkien.cxtvn.com/6685-dien-tro-0805-1-thong-so-tu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
- R17, R40, R5, R55, R76, R79, R8, R82, R9: value 10k -> 10kR; footprint (none) -> Resistor_SMD:R_0805_2012Metric; Link to Buy (none) -> https://linhkien.cxtvn.com/9909-dien-tro-0805-05-18w-10-chi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
- R4: footprint (none) -> Resistor_SMD:R_0402_1005Metric; Link to Buy (none) -> https://linhkien.cxtvn.com/7030-dien-tro-0402-1-thong-so-tu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
- R53, R54: value 100R -> 120R; footprint (none) -> Resistor_SMD:R_0402_1005Metric; Link to Buy (none) -> https://linhkien.cxtvn.com/7030-dien-tro-0402-1-thong-so-tu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
- R56, R60: value 100 -> 120R; footprint (none) -> Resistor_SMD:R_0402_1005Metric; Link to Buy (none) -> https://linhkien.cxtvn.com/7030-dien-tro-0402-1-thong-so-tu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
- R57, R58, R59: value 4.7k -> 4.7kR; footprint Resistor_SMD:R_0402_1005Metric_Pad0.72x0.64mm_HandSolder -> Resistor_SMD:R_0805_2012Metric; Link to Buy (none) -> https://linhkien.cxtvn.com/6337-dien-tro-0805-1-thong-so-tu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
- R74, R77: value 470R -> 220R; footprint (none) -> Resistor_SMD:R_0805_2012Metric; Link to Buy (none) -> https://linhkien.cxtvn.com/1958-dien-tro-0805-5-thong-so-10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
- R75, R78, R81: value 3.3k -> 3.3kR; footprint (none) -> Resistor_SMD:R_0805_2012Metric; Link to Buy (none) -> https://linhkien.cxtvn.com/4177-dien-tro-0805-1-thong-so-tu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
- R80: footprint (none) -> Resistor_SMD:R_0805_2012Metric; Link to Buy (none) -> https://linhkien.cxtvn.com/2345-dien-tro-470r-0805-1-100c.h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
- U1, U10, U6: LCSC Part (none) -> C119091; Link to Buy (none) -> https://linhkienchatluong.vn/urlltv/ltv357-ltv357t-sop-4-ch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; MPN (none) -> LTV-357T; Manufacturer (none) -> Lite-On
- U3: LCSC Part (none) -> C18148; Link to Buy (none) -> https://linhkienthuduc.com/san-pham/max3485csa-rs485-ic-soi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; MPN (none) -> MAX3485CSA; Manufacturer (none) -> Maxim (Analog Devices)
Connections:
- net +3V3: now also U12.5 (VIO)
- net +5V: now also U12.3 (VCC)
- net CAN_H: now also D9.2 (A2), U12.7 (CANH)
- net CAN_L: now also D9.1 (A1), U12.6 (CANL)
- net DO1_SINK: now also Q1.3 (D)
- net DO2_SINK: now also Q6.3 (D)
- net DO3_SINK: now also Q7.3 (D)
- net GND: now also D10.2 (A), D11.2 (A), D16.2 (A), D18.2 (A), D24.2 (A), D9.3 (common), Q1.2 (S), Q11.2 (S), Q12.2 (S), Q6.2 (S), Q7.2 (S), U12.2 (GND)
- net SW1_SENSE_N: now also Q11.3 (D)
- net SW2_SENSE_N: now also Q12.3 (D)
- net at R79.2, U6.3: now also D11.1 (K), Q6.1 (G)
- net at R53.2: now also U12.1 (TXD)
- net at C33.2, R12.2, R13.1: now also D18.1 (K), Q11.1 (G)
- net at C35.2, R38.2, R39.1: now also D24.1 (K), Q12.1 (G)
- net at R82.2, U10.3: now also D16.1 (K), Q7.1 (G)
- net at R76.2, U1.3: now also D10.1 (K), Q1.1 (G)
- net at R55.1: now also U12.8 (S)
- net at R54.2: now also U12.4 (RXD)
Other:
- moved on the sheet: C35, C36, C40, D1, D23, D5, R13, R38, R39, R40, R74, R75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
