File: Hardware/Current_Sensing.kicad_sch (KiCad schematic)
At the start: 2 parts, among them U11 INA241A2IDDFR

Commit message: feat: update buy link, footprint
Parts:
- C28: value 100nF -> 100nF 50V; footprint (none) -> Capacitor_SMD:C_0805_2012Metric; Link to Buy (none) -> https://linhkien.cxtvn.com/1976-tu-khong-phan-cuc-0805.html
- U11: Link to Buy (none) -> https://www.lcsc.com/product-detail/C5240853.html?s_z=n_q_x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
Changed lines of the file:
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@@
 		(lib_id "Device:C_Small")
 		(at 147.32 105.41 90)
-		(unit 1)
-		(body_style 1)
-		(exclude_from_sim no)
-		(in_bom yes)
-		(on_board yes)
-		(in_pos_files yes)
-		(dnp no)
-		(fields_autoplaced yes)
+		(mirror x)
+		(unit 1)
+		(body_style 1)
+		(exclude_from_sim no)
+		(in_bom yes)
+		(on_board yes)
+		(in_pos_files yes)
+		(dnp no)
 		(property "Reference" "C28"
-			(at 147.3263 99.06 90)
-			(show_name no)
-			(do_not_autoplace no)
-			(effects
-				(font
-					(size 1.27 1.27)
-				)
-			)
-		)
-		(property "Value" "100nF"
-			(at 147.3263 101.6 90)
-			(show_name no)
-			(do_not_autoplace no)
-			(effects
-				(font
-					(size 1.27 1.27)
-				)
-			)
-		)
-		(property "Footprint" ""
+			(at 149.098 108.712 90)
+			(show_name no)
+			(do_not_autoplace no)
+			(effects
+				(font
+					(size 1.27 1.27)
+				)
+				(justify left)
+			)
+		)
+		(property "Value" "100nF 50V"
+			(at 152.146 111.252 90)
+			(show_name no)
+			(do_not_autoplace no)
+			(effects
+				(font
+					(size 1.27 1.27)
+				)
+				(justify left)
+			)
+		)
+		(property "Footprint" "Capacitor_SMD:C_0805_2012Metric"
 			(at 147.32 105.41 0)
 			(hide yes)
@@
 		(property "Description" "Unpolarized capacitor, small symbol"
 			(at 147.32 105.41 0)
+			(hide yes)
+			(show_name no)
+			(do_not_autoplace no)
+			(effects
+				(font
+					(size 1.27 1.27)
+				)
+			)
+		)
+		(property "Link to Buy" "https://linhkien.cxtvn.com/1976-tu-khong-phan-cuc-0805.html"
+			(at 31.75 17.78 0)
 			(hide yes)
 			(show_name no)
@@
 			)
 		)
-		(property "Description" "High- and Low-Side, Bidirectional, Zero-Drift, Current-Sense Amplifier With Enhanced PWM Rejection, 20V/V, ±0.01% Gain Accuracy, ±10 μV Offset Voltage, SOT-23-8"
+		(property "Description" "NA241x –5 V to 110 V, Bidirectional, Ultra-Precise Current Sense Amplifier WithEnhanced PWM Rejection"
 			(at 156.21 92.71 0)
 			(hide yes)
+			(show_name no)
+			(do_not_autoplace no)
+			(effects
+				(font
+					(size 1.27 1.27)
+				)
+			)
+		)
+		(property "Link to Buy" "https://www.lcsc.com/product-detail/C5240853.html?s_z=n_q_x_INA241A2IDDFR"
+			(at 156.21 92.71 0)
+			(hide yes)

Commit message: feat: update schematic with new components for communication interfaces and export BOM list
Parts:
- C28: value 100nF 50V -> 100nF
Changed lines of the file:
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@@
 			)
 		)
-		(property "Value" "100nF 50V"
+		(property "Value" "100nF"
 			(at 152.146 111.252 90)
 			(show_name no)
