File: Hardware/MCU_Control.kicad_sch (KiCad schematic)
At the start: 29 parts, among them J1 USB2.0_16P, Q3 BC817, Q4 BC817, SW1 ENABLE, U4 ESP32-WROOM-32E, U5 USBLC6-2SC6, U7 CP2102N-A02-GQFN20

Commit message: feat: update schematic with new components for communication interfaces and export BOM list
Parts:
- removed C21: 10uF, symbol Device:C_Polarized
- removed C23: 4.7u, Footprints:T491A, symbol T491A106K010AT7280:T491A106K010AT7280
- removed D9: 1N5817, Diode_THT:D_DO-41_SOD81_P10.16mm_Horizontal, symbol Diode:1N5817
- added C21: 10uF, Capacitor_SMD:C_0805_2012Metric, symbol Device:C_Small
- added C23: 4.7uF, Capacitor_SMD:C_1206_3216Metric, symbol SparkFun-Capacitor:C
- C14: value 1u -> 1uF; Link to Buy (none) -> https://linhkien.cxtvn.com/1976-tu-khong-phan-cuc-0805.html
- C15, C24: value 0.1u -> 100nF; Link to Buy (none) -> https://linhkien.cxtvn.com/1976-tu-khong-phan-cuc-0805.html
- C22: footprint (none) -> Capacitor_SMD:C_0805_2012Metric; Link to Buy (none) -> https://linhkien.cxtvn.com/1976-tu-khong-phan-cuc-0805.html
- C25: value 10u -> 10uF; footprint Footprints:T491A -> Capacitor_SMD:C_0805_2012Metric; Link to Buy (none) -> https://linhkien.cxtvn.com/1976-tu-khong-phan-cuc-0805.html
- C26: value 1u -> 1uF; footprint Capacitor_SMD:C_0603_1608Metric -> Capacitor_SMD:C_0805_2012Metric; Link to Buy (none) -> https://linhkien.cxtvn.com/1976-tu-khong-phan-cuc-0805.html
- D12: value GREEN -> LED_G; Link to Buy (none) -> https://linhkienchatluong.vn/urlled-dan-0603-smd/led-dan-06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
- D13: value RED -> LED_R; Link to Buy (none) -> https://linhkienchatluong.vn/urlled-dan-0603-smd/led-dan-06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
- F2: value Fuse 1A -> Fuse; LCSC Part (none) -> C66453; Link to Buy (none) -> https://linhkienthuduc.com/san-pham/nsmd100-cau-chi-tu-phuc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; MPN (none) -> nSMD100
- J1: Link to Buy (none) -> https://linhkienthuduc.com/san-pham/cong-usb-type-c-16-chan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; MPN (none) -> USB4105-GF-A; Manufacturer (none) -> GCT (Global Connector Technology)
- Q3, Q4: Link to Buy (none) -> https://linhkien.cxtvn.com/5979-bc817-40-transistor-npn-45v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
- R21, R22: value 5.1k -> 5.1kR; footprint Resistor_SMD:R_0402_1005Metric_Pad0.72x0.64mm_HandSolder -> Resistor_SMD:R_0805_2012Metric; Link to Buy (none) -> https://linhkien.cxtvn.com/6337-dien-tro-0805-1-thong-so-tu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
- R23: value 22K1 -> 22kR; Link to Buy (none) -> https://linhkien.cxtvn.com/6337-dien-tro-0805-1-thong-so-tu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
- R24: value 47K5 -> 47kR; Link to Buy (none) -> https://linhkienchatluong.vn/urlloai-0805-sai-so-1/dien-tro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
- R25: value 2.2k -> 2.2kR; Link to Buy (none) -> https://linhkien.cxtvn.com/6337-dien-tro-0805-1-thong-so-tu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
- R26, R27: value 1K -> 1kR; footprint Resistor_SMD:R_0402_1005Metric_Pad0.72x0.64mm_HandSolder -> Resistor_SMD:R_0805_2012Metric; Link to Buy (none) -> https://linhkien.cxtvn.com/6337-dien-tro-0805-1-thong-so-tu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
- R28: value 10K -> 10kR; footprint Resistor_SMD:R_0402_1005Metric_Pad0.72x0.64mm_HandSolder -> Resistor_SMD:R_0805_2012Metric; Link to Buy (none) -> https://linhkien.cxtvn.com/9909-dien-tro-0805-05-18w-10-chi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
- R33, R34: value 10K -> 10kR; Link to Buy (none) -> https://linhkien.cxtvn.com/9909-dien-tro-0805-05-18w-10-chi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
- SW1: LCSC Part (none) -> C231329; Link to Buy (none) -> https://linhkien.cxtvn.com/10278-b3u-1000p-nut-nhan-smd-2p-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; MPN (none) -> B3U-1000P; Manufacturer (none) -> Omron
- U4: Link to Buy (none) -> https://linhkienthuduc.com/san-pham/wifi-ble-module-esp32-e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; MPN (none) -> ESP32-WROOM-32E; Manufacturer (none) -> Espressif
- U5: LCSC Part (none) -> C7519; Link to Buy (none) -> https://linhkien.cxtvn.com/6071-usblc6-2sc6-tvs-diode-525v-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; MPN (none) -> USBLC6-2SC6; Manufacturer (none) -> STMicroelectronics
- U7: LCSC Part (none) -> C969913; Link to Buy (none) -> https://ic-vietnam.com.vn/mach-tich-hop-ic-cp2102n-a02-gqfn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; MANUFACTURER Silicon Laboratories -> (none); MPN (none) -> CP2102N-A02-GQFN20R; Manufacturer (none) -> Silicon Labs
Connections:
- net +3V3: now also C23.1
- net GND: now also C21.2, C23.2
- net V_USB: now also F2.2, C21.1
