File: Hardware/robot-hv-charge-controller.kicad_pcb (KiCad board)
At the start: 2 copper layers, 10 parts, among them J2 XT30PW-M, J3 XT30PW-M, M1 IPB107N20N3GATMA1, M2 IPB107N20N3GATMA1, M3 IPB107N20N3GATMA1, M4 IPB107N20N3GATMA1, M5 IPB107N20N3GATMA1, M6 IPB107N20N3GATMA1, M7 IPB107N20N3GATMA1, M8 IPB107N20N3GATMA1

Commit message: feat: update components link, footprint and package
Parts:
- removed J2, J3: XT30PW-M, Connector_AMASS:AMASS_XT30PW-M_1x02_P2.50mm_Horizontal
- removed M1, M2, M3, M4, M5, M6, M7, M8: IPB107N20N3GATMA1, IPB107N20N3GATMA1:PG-TO263-3 _10P06X8P98_INF-M
- added C14: 1u, Capacitor_SMD:C_0805_2012Metric, F.Cu at (375.6, 107.4)
- added C15: 0.1u, Capacitor_SMD:C_0805_2012Metric, F.Cu at (375.6, 110.4)
- added C2: 100nF 50V, Capacitor_SMD:C_0805_2012Metric, F.Cu at (224.9, 46.0)
- added C24: 0.1u, Capacitor_SMD:C_0805_2012Metric, F.Cu at (375.6, 113.4)
- added C26: 1u, Capacitor_SMD:C_0603_1608Metric, F.Cu at (351.7, 111.4)
- added C3: 47uF 50V, Capacitor_SMD:CP_Elec_6.3x7.7, F.Cu at (225.0, 58.0)
- added D1: FR107, Diode_THT:D_DO-35_SOD27_P7.62mm_Horizontal, F.Cu at (406.9, 65.0)
- added D12: GREEN, LED_SMD:LED_0603_1608Metric, F.Cu at (396.2, 107.1)
- added D13: RED, LED_SMD:LED_0603_1608Metric, F.Cu at (396.2, 109.7)
- added D14: GREEN, LED_SMD:LED_0603_1608Metric, F.Cu at (402.5, 106.8)
- added D15: BAV21W, Diode_THT:D_DO-35_SOD27_P7.62mm_Horizontal, F.Cu at (402.0, 111.8)
- added D19: ESD, Diode_SMD:D_SOD-923, F.Cu at (401.9, 86.5)
- added D2: 1N4148W, Diode_SMD:D_SOD-123, F.Cu at (225.7, 38.0)
- added D20: LED_G, LED_SMD:LED_0603_1608Metric, F.Cu at (418.2, 80.5)
- added D21: LED_Y, LED_SMD:LED_0603_1608Metric, F.Cu at (418.2, 83.1)
- added D22: LED_Y, LED_SMD:LED_0603_1608Metric, F.Cu at (418.2, 85.7)
- added D23: ESD, Diode_SMD:D_SOD-923, F.Cu at (401.9, 88.4)
- added D25: 1N914, Diode_THT:D_DO-35_SOD27_P7.62mm_Horizontal, F.Cu at (406.9, 75.7)
- added D26: 1N914, Diode_THT:D_DO-35_SOD27_P7.62mm_Horizontal, F.Cu at (406.9, 79.2)
- added D3: SS34, Diode_SMD:D_SMA, F.Cu at (404.5, 94.1)
- added D4: SMAJ36A, Diode_SMD:D_SMA, F.Cu at (404.5, 98.6)
- added D5: FR107, Diode_THT:D_DO-35_SOD27_P7.62mm_Horizontal, F.Cu at (406.9, 68.6)
- added D6: FR107, Diode_THT:D_DO-35_SOD27_P7.62mm_Horizontal, F.Cu at (406.9, 72.1)
- added D7: FR107, Diode_SMD:Nexperia_CFP3_SOD-123W, F.Cu at (235.0, 50.0)
- added D8: SS34, Diode_SMD:D_SMA, F.Cu at (404.5, 103.2)
- added D9: 1N5817, Diode_THT:D_DO-41_SOD81_P10.16mm_Horizontal, F.Cu at (346.4, 108.0)
- added F2: Fuse 1A, Fuse:Fuse_1206_3216Metric, F.Cu at (385.5, 111.9)
- added F3: Fuse 1A, Fuse:Fuse_1206_3216Metric, F.Cu at (411.4, 100.1)
- added J1: USB2.0_16P, Connector_USB:USB_C_Receptacle_GCT_USB4105-xx-A_16P_TopMnt_Horizontal, F.Cu at (364.3, 111.1)
- added J5: XT60PW-M, XT60PW-M:AMASS_XT60PW-M, F.Cu at (354.9, 50.1)
- added J6: XT60PW-M, XT60PW-M:AMASS_XT60PW-M, F.Cu at (373.8, 50.1)
- added J7: XT60PW-M, XT60PW-M:AMASS_XT60PW-M, F.Cu at (392.6, 50.1)
- added Q1: BCX56-16, Package_TO_SOT_SMD:SOT-23, F.Cu at (402.9, 65.5)
- added Q11: MMBT3904, Package_TO_SOT_SMD:SOT-23, F.Cu at (402.9, 78.8)
- added Q12: MMBT3904, Package_TO_SOT_SMD:SOT-23, F.Cu at (402.9, 83.3)
- added Q3: BC817, Package_TO_SOT_SMD:SOT-23, F.Cu at (380.3, 108.1)
- added Q4: BC817, Package_TO_SOT_SMD:SOT-23, F.Cu at (380.3, 112.5)
- added Q6: BCX56-16, Package_TO_SOT_SMD:SOT-23, F.Cu at (402.9, 69.9)
- added Q7: BCX56-16, Package_TO_SOT_SMD:SOT-23, F.Cu at (402.9, 74.4)
- added Q8: BC817-40, Package_TO_SOT_SMD:SOT-23, F.Cu at (234.9, 66.0)
- added R21: 5.1k, Resistor_SMD:R_0402_1005Metric_Pad0.72x0.64mm_HandSolder, F.Cu at (371.7, 106.8)
- added R22: 5.1k, Resistor_SMD:R_0402_1005Metric_Pad0.72x0.64mm_HandSolder, F.Cu at (371.7, 108.8)
- added R23: 22K1, Resistor_SMD:R_0805_2012Metric, F.Cu at (396.3, 64.7)
- added R24: 47K5, Resistor_SMD:R_0805_2012Metric, F.Cu at (396.3, 67.7)
- added R25: 2.2k, Resistor_SMD:R_0805_2012Metric, F.Cu at (396.3, 70.6)
- added R26: 1K, Resistor_SMD:R_0402_1005Metric_Pad0.72x0.64mm_HandSolder, F.Cu at (371.7, 110.8)
- added R27: 1K, Resistor_SMD:R_0402_1005Metric_Pad0.72x0.64mm_HandSolder, F.Cu at (371.7, 112.8)
- added R28: 10K, Resistor_SMD:R_0402_1005Metric_Pad0.72x0.64mm_HandSolder, F.Cu at (371.7, 114.8)
- added R33: 10K, Resistor_SMD:R_0805_2012Metric, F.Cu at (396.3, 73.6)
- added R34: 10K, Resistor_SMD:R_0805_2012Metric, F.Cu at (396.3, 76.5)
- added R37: 4.7k, Resistor_SMD:R_0402_1005Metric_Pad0.72x0.64mm_HandSolder, F.Cu at (406.1, 106.5)
- added R41: 1.8mR, CSS2H_2512R_1L00F:RES_1L00x_BRN, F.Cu at (404.7, 116.1)
- added R57: 4.7k, Resistor_SMD:R_0402_1005Metric_Pad0.72x0.64mm_HandSolder, F.Cu at (421.8, 80.2)
- added R58: 4.7k, Resistor_SMD:R_0402_1005Metric_Pad0.72x0.64mm_HandSolder, F.Cu at (421.8, 82.2)
- added R59: 4.7k, Resistor_SMD:R_0402_1005Metric_Pad0.72x0.64mm_HandSolder, F.Cu at (421.8, 84.2)
- added R83: 470R, Resistor_SMD:R_0805_2012Metric, F.Cu at (225.9, 77.0)
- added R84: 3.3k, Resistor_SMD:R_0805_2012Metric, F.Cu at (242.9, 60.0)
- added R85: 10k, Resistor_SMD:R_0805_2012Metric, F.Cu at (236.9, 77.0)
- added SW1: ENABLE, Button_Switch_SMD:SW_SPST_B3U-1000P, F.Cu at (385.7, 108.0)
- added U1: LTV-357T, Package_SO:SO-4_4.4x3.6mm_P2.54mm, F.Cu at (421.1, 66.0)
- added U10: LTV-357T, Package_SO:SO-4_4.4x3.6mm_P2.54mm, F.Cu at (421.1, 76.6)
- added U11: INA241A2IDDFR, Package_TO_SOT_SMD:SOT-23-8, F.Cu at (415.8, 112.4)
- added U12: MCP2542FDxMF, Package_DFN_QFN:DFN-8-1EP_3x3mm_P0.65mm_EP1.55x2.4mm, F.Cu at (423.3, 87.5)
- added U13: LTV-354T, Package_SO:SO-4_4.4x3.6mm_P2.54mm, F.Cu at (251.0, 72.0)
- added U2: RT9013-33GB, Package_TO_SOT_SMD:SOT-23-5, F.Cu at (411.1, 104.2)
- added U3: MAX3485, Package_SO:SOIC-8_3.9x4.9mm_P1.27mm, F.Cu at (409.6, 84.4)
- added U4: ESP32-WROOM-32E, RF_Module:ESP32-WROOM-32E, F.Cu at (369.3, 91.8)
- added U5: USBLC6-2SC6, Package_TO_SOT_SMD:SOT-23-6, F.Cu at (347.1, 112.5)
- added U6: LTV-357T, Package_SO:SO-4_4.4x3.6mm_P2.54mm, F.Cu at (421.1, 71.3)
- added U7: CP2102N-A02-GQFN20, Package_DFN_QFN:SiliconLabs_QFN-20-1EP_3x3mm_P0.5mm_EP1.8x1.8mm, F.Cu at (391.4, 108.6)
- added U8: HF116F-80/24-1HTF, HF116F-80-12-24-1HTF:RELAY-TH_HF116F-80-XX-1HTF, F.Cu at (231.4, 107.8)
- added U9: LV14340DDAR, LV14340DDAR:SOIC8_DDA_TEX, F.Cu at (412.8, 95.2)
Other:
- board text added: "Main_Relay_Control"

Commit message: feat: update buy link, footprint
Parts:
- added C28: 100nF 50V, Capacitor_SMD:C_0805_2012Metric, F.Cu at (156.7, 94.0)
- added C29: 100nF 50V, Capacitor_SMD:C_0805_2012Metric, F.Cu at (165.1, 43.0)
- added R42: 10k, Resistor_SMD:R_0805_2012Metric, F.Cu at (156.6, 41.0)
- added R43: 150k, Resistor_SMD:R_0805_2012Metric, F.Cu at (157.0, 51.0)
- added R44: 150k, Resistor_SMD:R_0805_2012Metric, F.Cu at (166.0, 51.0)
- added R45: 150k, Resistor_SMD:R_0805_2012Metric, F.Cu at (156.6, 58.0)
- added R46: 18k, Resistor_SMD:R_0805_2012Metric, F.Cu at (165.0, 58.0)
- D15: footprint Diode_THT:D_DO-35_SOD27_P7.62mm_Horizontal -> Diode_SMD:D_SOD-123
- moved U11 249.5 mm to (167.0, 94.0)
- moved D15 248.8 mm to (156.7, 71.0)
- moved R41 242.2 mm to (167.0, 70.0)
Other:
- board text added: "Current_Sensing"
- board text added: "Output_Protection_and_Sensing"

Commit message: feat: update footprint power supply
Parts:
- added C10: 1u, Capacitor_SMD:C_0805_2012Metric, F.Cu at (105.1, 50.0)
- added C11: 100n, Capacitor_SMD:C_0805_2012Metric, F.Cu at (109.5, 38.0)
- added C12: 100u, Capacitor_SMD:CP_Elec_5x5.4, F.Cu at (107.0, 62.0)
- added C13: 33pF, Capacitor_SMD:C_0805_2012Metric, F.Cu at (109.5, 41.0)
- added C16: 22uF, Capacitor_SMD:C_0805_2012Metric, F.Cu at (109.5, 44.0)
- added C17: 22uF, Capacitor_SMD:C_0805_2012Metric, F.Cu at (109.5, 47.0)
- added C18: 100nF, Capacitor_SMD:C_0805_2012Metric, F.Cu at (109.5, 50.0)
- added C19: 100nF, Capacitor_SMD:C_0805_2012Metric, F.Cu at (114.0, 38.0)
- added C20: 1uF, Capacitor_SMD:C_0805_2012Metric, F.Cu at (114.0, 41.0)
- added C27: 10uF, Capacitor_SMD:C_0805_2012Metric, F.Cu at (114.0, 44.0)
- added C6: 22nF, Capacitor_SMD:C_0805_2012Metric, F.Cu at (105.1, 38.0)
- added C7: 100nF 50V, Capacitor_SMD:C_0805_2012Metric, F.Cu at (105.1, 41.0)
- added C8: 10u, Capacitor_SMD:C_0805_2012Metric, F.Cu at (105.1, 44.0)
- added C9: 100n, Capacitor_SMD:C_0805_2012Metric, F.Cu at (105.1, 47.0)
- added L2: 6.8uH, Inductor_SMD:L_SXN_SMDRI73, F.Cu at (121.0, 41.0)
- added R10: 49.9, Resistor_SMD:R_0603_1608Metric, F.Cu at (118.2, 46.8)
- added R11: 68k, Resistor_SMD:R_0603_1608Metric, F.Cu at (118.2, 49.3)
- added R48: 12k, Resistor_SMD:R_0603_1608Metric, F.Cu at (118.2, 51.8)
- D4: value SMAJ36A -> SMAJ36CA
- moved F3 305.3 mm to (106.4, 85.0)
- moved D3 298.1 mm to (107.0, 75.0)
- moved U9 295.6 mm to (119.0, 63.0)
- moved U2 293.3 mm to (119.1, 76.0)
- moved R37 288.2 mm to (118.6, 87.0)
- moved D8 279.3 mm to (130.0, 52.0)
- moved D4 276.7 mm to (130.0, 64.0)
- moved D14 275.4 mm to (128.8, 76.0)
Other:
- board text added: "Auxiliary_Power_supply"

Commit message: feat: update schematic with new components for communication interfaces and export BOM list
Parts:
- removed the Q11 at (402.9, 78.8)
- added C21: 10uF, Capacitor_SMD:C_0805_2012Metric, F.Cu at (-137.8, 116.7)
- added C22: 100nF, Capacitor_SMD:C_0805_2012Metric, F.Cu at (-148.8, 126.7)
- added C23: 4.7uF, Capacitor_SMD:C_1206_3216Metric, F.Cu at (-137.3, 124.7)
- added C25: 10uF, Capacitor_SMD:C_0805_2012Metric, F.Cu at (-145.8, 116.7)
- added C32: 33pF, Capacitor_SMD:C_0805_2012Metric, F.Cu at (-251.5, 40.9)
- added C33: 100nF, Capacitor_SMD:C_0805_2012Metric, F.Cu at (-251.5, 45.4)
- added C34: 100nF, Capacitor_SMD:C_0805_2012Metric, F.Cu at (-252.6, 51.7)
- added C35: 100nF, Capacitor_SMD:C_0805_2012Metric, F.Cu at (-247.6, 51.7)
- added C36: 100nF, Capacitor_SMD:C_0805_2012Metric, F.Cu at (-242.6, 50.7)
- added C37: 33pF, Capacitor_SMD:C_0805_2012Metric, F.Cu at (-237.6, 45.7)
- added C38: 100nF, Capacitor_SMD:C_0805_2012Metric, F.Cu at (-242.6, 45.7)
- added C39: 10uF, Capacitor_SMD:C_0805_2012Metric, F.Cu at (-226.8, 54.7)
- added C4: 100nF, Capacitor_SMD:C_0805_2012Metric, F.Cu at (-251.5, 35.9)
- added C40: 100nF, Capacitor_SMD:C_0805_2012Metric, F.Cu at (-246.6, 45.7)
- added D10: BZT52C12, Diode_SMD:D_SOD-123, F.Cu at (-218.2, 48.0)
- added D11: BZT52C12, Diode_SMD:D_SOD-123, F.Cu at (-226.2, 82.0)
- added D16: BZT52C12, Diode_SMD:D_SOD-123, F.Cu at (-219.2, 68.0)
- added D17: BZT52C12, Diode_SMD:D_SOD-123, F.Cu at (-97.2, 56.0)
- added D18: BZT52C12, Diode_SMD:D_SOD-123, F.Cu at (-251.2, 87.0)
- added D24: BZT52C12, Diode_SMD:D_SOD-123, F.Cu at (-243.2, 87.0)
- added F2: Fuse, Fuse:Fuse_1206_3216Metric, F.Cu at (-137.2, 130.7)
- added J10: Screw_01x02, TerminalBlock_Phoenix:TerminalBlock_Phoenix_MKDS-1,5-2_1x02_P5.00mm_Horizontal, F.Cu at (-302.1, 169.0)
- added J11: Screw_01x02, TerminalBlock_Phoenix:TerminalBlock_Phoenix_MKDS-1,5-2_1x02_P5.00mm_Horizontal, F.Cu at (-290.0, 169.0)
- added J12: Screw_01x02, TerminalBlock_Phoenix:TerminalBlock_Phoenix_MKDS-1,5-2_1x02_P5.00mm_Horizontal, F.Cu at (-302.1, 181.1)
- added J13: Screw_01x02, TerminalBlock_Phoenix:TerminalBlock_Phoenix_MKDS-1,5-2_1x02_P5.00mm_Horizontal, F.Cu at (-290.0, 181.1)
- added J2: UART_CONN, Connector_PinHeader_2.54mm:PinHeader_1x04_P2.54mm_Horizontal, F.Cu at (-278.3, 141.3)
- added J3: XT30PW-M, XT30PW-M:AMASS_XT30PW-M, F.Cu at (-277.6, 120.0)
- added J4: Screw_01x02, TerminalBlock_Phoenix:TerminalBlock_Phoenix_MKDS-1,5-2_1x02_P5.00mm_Horizontal, F.Cu at (-302.1, 144.7)
- added J8: Screw_01x02, TerminalBlock_Phoenix:TerminalBlock_Phoenix_MKDS-1,5-2_1x02_P5.00mm_Horizontal, F.Cu at (-302.1, 156.9)
- added J9: Screw_01x02, TerminalBlock_Phoenix:TerminalBlock_Phoenix_MKDS-1,5-2_1x02_P5.00mm_Horizontal, F.Cu at (-290.0, 156.9)
- added Q11: SI2308BDS, Package_TO_SOT_SMD:SOT-23, F.Cu at (-222.2, 74.0)
- added Q11: MMBT3904, Package_TO_SOT_SMD:SOT-23, F.Cu at (-226.8, 62.7)
- added R12: 4.7kR, Resistor_SMD:R_0805_2012Metric, F.Cu at (-228.4, 48.7)
- added R13: 150kR, Resistor_SMD:R_0805_2012Metric, F.Cu at (-224.4, 48.7)
- added R17: 10kR, Resistor_SMD:R_0805_2012Metric, F.Cu at (-244.6, 35.6)
- added R38: 4.7kR, Resistor_SMD:R_0805_2012Metric, F.Cu at (-244.6, 40.1)
- added R39: 150kR, Resistor_SMD:R_0805_2012Metric, F.Cu at (-229.1, 35.1)
- added R4: 120R, Resistor_SMD:R_0402_1005Metric, F.Cu at (-247.8, 35.6)
- added R40: 10kR, Resistor_SMD:R_0805_2012Metric, F.Cu at (-223.6, 40.1)
- added R5: 10kR, Resistor_SMD:R_0805_2012Metric, F.Cu at (-247.8, 40.1)
- added R53: 120R, Resistor_SMD:R_0402_1005Metric, F.Cu at (-223.6, 42.1)
- added R54: 120R, Resistor_SMD:R_0402_1005Metric, F.Cu at (-223.6, 44.1)
- added R55: 10kR, Resistor_SMD:R_0805_2012Metric, F.Cu at (-241.3, 35.6)
- added R56: 120R, Resistor_SMD:R_0402_1005Metric, F.Cu at (-241.3, 40.1)
- added R6: 1kR, Resistor_SMD:R_0805_2012Metric, F.Cu at (-270.6, 165.0)
- added R60: 120R, Resistor_SMD:R_0402_1005Metric, F.Cu at (-225.8, 35.1)
- added R7: 1kR, Resistor_SMD:R_0805_2012Metric, F.Cu at (-273.1, 159.0)
- added R74: 220R, Resistor_SMD:R_0805_2012Metric, F.Cu at (-228.0, 40.1)
- added R75: 3.3kR, Resistor_SMD:R_0805_2012Metric, F.Cu at (-228.0, 42.1)
- added R76: 10kR, Resistor_SMD:R_0805_2012Metric, F.Cu at (-228.0, 44.1)
- added R77: 220R, Resistor_SMD:R_0805_2012Metric, F.Cu at (-238.0, 35.6)
- added R78: 3.3kR, Resistor_SMD:R_0805_2012Metric, F.Cu at (-238.0, 40.1)
- added R79: 10kR, Resistor_SMD:R_0805_2012Metric, F.Cu at (-222.6, 35.1)
- added R8: 10kR, Resistor_SMD:R_0805_2012Metric, F.Cu at (-232.4, 35.1)
- added R80: 470R, Resistor_SMD:R_0805_2012Metric, F.Cu at (-232.6, 40.1)
- added R81: 3.3kR, Resistor_SMD:R_0805_2012Metric, F.Cu at (-232.6, 42.1)
- added R82: 10kR, Resistor_SMD:R_0805_2012Metric, F.Cu at (-232.6, 44.1)
- added R9: 10kR, Resistor_SMD:R_0805_2012Metric, F.Cu at (-232.7, 47.9)
- C10, C14: value 1u -> 1uF
- C11, C9: value 100n -> 100nF
- C12: value 100u -> 100uF
- C15, C24: value 0.1u -> 100nF
- C2, C28, C29, C7: value 100nF 50V -> 100nF
- C26: value 1u -> 1uF; footprint Capacitor_SMD:C_0603_1608Metric -> Capacitor_SMD:C_0805_2012Metric
- C3: value 47uF 50V -> 47uF
- C8: value 10u -> 10uF
- D1, D5, D6: value FR107 -> RS1M; footprint Diode_THT:D_DO-35_SOD27_P7.62mm_Horizontal -> Diode_SMD:D_SOD-123
- D12, D14: value GREEN -> LED_G
- D13: value RED -> LED_R
- D19, D23: value ESD -> PESD5Z3.3; footprint Diode_SMD:D_SOD-923 -> Diode_SMD:D_SOD-323
- D25, D26: value 1N914 -> 1N4148W; footprint Diode_THT:D_DO-35_SOD27_P7.62mm_Horizontal -> Diode_SMD:D_SOD-123
- D7: value FR107 -> RS1M; footprint Diode_SMD:Nexperia_CFP3_SOD-123W -> Diode_SMD:D_SOD-123
- D9: value 1N5817 -> SM712; footprint Diode_THT:D_DO-41_SOD81_P10.16mm_Horizontal -> Package_TO_SOT_SMD:SOT-23
- F3: value Fuse 1A -> Fuse
- J6: value XT60PW-M -> Screw_01x02; footprint XT60PW-M:AMASS_XT60PW-M -> TerminalBlock_Phoenix:TerminalBlock_Phoenix_MKDS-1,5-2_1x02_P5.00mm_Horizontal
- Q1, Q6, Q7: value BCX56-16 -> SI2308BDS
- Q12: value MMBT3904 -> SI2308BDS
- Q8: value BC817-40 -> SI2308BDS
- R10: value 49.9 -> 49.9R
- R11: value 68k -> 68kR
- R21, R22: value 5.1k -> 5.1kR; footprint Resistor_SMD:R_0402_1005Metric_Pad0.72x0.64mm_HandSolder -> Resistor_SMD:R_0805_2012Metric
- R23: value 22K1 -> 22kR
- R24: value 47K5 -> 47kR
- R25: value 2.2k -> 2.2kR
- R26, R27: value 1K -> 1kR; footprint Resistor_SMD:R_0402_1005Metric_Pad0.72x0.64mm_HandSolder -> Resistor_SMD:R_0805_2012Metric
- R28: value 10K -> 10kR; footprint Resistor_SMD:R_0402_1005Metric_Pad0.72x0.64mm_HandSolder -> Resistor_SMD:R_0805_2012Metric
- R33, R34: value 10K -> 10kR
- R37, R57, R58, R59: value 4.7k -> 4.7kR; footprint Resistor_SMD:R_0402_1005Metric_Pad0.72x0.64mm_HandSolder -> Resistor_SMD:R_0805_2012Metric
- R42, R85: value 10k -> 10kR
- R43, R44, R45: value 150k -> 150kR
- R46: value 18k -> 18kR
- R48: value 12k -> 12kR; footprint Resistor_SMD:R_0603_1608Metric -> Resistor_SMD:R_0805_2012Metric
- R83: value 470R -> 220R
- R84: value 3.3k -> 3.3kR
- U12: value MCP2542FDxMF -> TJA1051T-3; footprint Package_DFN_QFN:DFN-8-1EP_3x3mm_P0.65mm_EP1.55x2.4mm -> Package_SO:SOIC-8_3.9x4.9mm_P1.27mm
- U13: value LTV-354T -> LTV-357T
- moved J6 670.5 mm to (-290.0, 144.7)
- moved D20 664.9 mm to (-246.7, 76.2)
- moved D21 664.9 mm to (-246.7, 78.8)
- moved D22 664.9 mm to (-246.7, 81.4)
- moved R57 664.9 mm to (-243.1, 75.9)
- moved R58 664.9 mm to (-243.1, 77.9)
- moved R59 664.9 mm to (-243.1, 79.9)
- moved U1 664.9 mm to (-243.8, 61.7)
- moved U10 664.9 mm to (-243.8, 72.4)
- moved U6 664.9 mm to (-243.8, 67.0)
- moved D26 658.6 mm to (-251.6, 74.1)
- moved D25 658.6 mm to (-251.6, 70.7)
- moved D6 658.6 mm to (-251.6, 67.4)
- moved D5 658.6 mm to (-251.6, 64.0)
- moved D1 658.6 mm to (-251.6, 60.7)
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Connections:
- net /IOUT_SENSE_ADC renamed /Current_Sensing/IOUT_SENSE_ADC
- net /MAIN_RELAY_EN renamed /MCU_Control/MAIN_RELAY_EN
- net /VOUT_SENSE_ADC renamed /MCU_Control/VOUT_SENSE_ADC
- D19 pad 1: /UART_EXT_TX_CONN -> /Communication_Interfaces/UART_EXT_TX_CONN
- D23 pad 1: /UART_EXT_RX_CONN -> /Communication_Interfaces/UART_EXT_RX_CONN
- D25 pad 1: /RS485_A -> /Communication_Interfaces/RS485_A
- D26 pad 1: /RS485_B -> /Communication_Interfaces/RS485_B
- D9 pad 1: V_USB -> /Communication_Interfaces/CAN_L
- D9 pad 2: Net-(D9-A) -> /Communication_Interfaces/CAN_H
- J6 pad 1: /Auxiliary_Power_Supply/VAUX_IN_P -> /Communication_Interfaces/RS485_B
- J6 pad 2: GND -> /Communication_Interfaces/RS485_A
- Q8 pad 1: Net-(Q8-B) -> Net-(D17-K)
- Q8 pad 2: GND -> /Main_Relay_Control/MAIN_RELAY_COIL_N
- Q8 pad 3: /Main_Relay_Control/MAIN_RELAY_COIL_N -> GND
- R85 pad 2: Net-(Q8-B) -> Net-(D17-K)
- U12 pad 6: /CAN_L -> /Communication_Interfaces/CAN_L
- U12 pad 7: /CAN_H -> /Communication_Interfaces/CAN_H
- U13 pad 1: Net-(R83-Pad2) -> Net-(R84-Pad1)
- U13 pad 2: GND -> Net-(D17-K)
- U13 pad 3: Net-(Q8-B) -> GND
- U13 pad 4: Net-(R84-Pad1) -> Net-(R83-Pad2)
- U3 pad 6: /RS485_A -> /Communication_Interfaces/RS485_A
- U3 pad 7: /RS485_B -> /Communication_Interfaces/RS485_B
Other:
- board text added: "Communication_Interfaces"
- board text added: "Connection"
- board text added: "MCU_Control"
