File: Hardware/Main_Relay_Control.kicad_sch (KiCad schematic)
At the start: 10 parts, among them Q8 BC817-40, U13 LTV-354T, U8 HF116F-80/24-1HTF

Commit message: fix: ground capacitor C3 C2
Parts:
- C3: footprint Capacitor_THT:CP_Radial_D6.3mm_P2.50mm -> Capacitor_SMD:CP_Elec_6.3x7.7
Changed lines of the file:
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@@
 			)
 		)
-		(property "Footprint" "Capacitor_THT:CP_Radial_D6.3mm_P2.50mm"
+		(property "Footprint" "Capacitor_SMD:CP_Elec_6.3x7.7"
 			(at 115.57 77.47 0)
 			(hide yes)

Commit message: feat: update components link, footprint and package
Parts:
- removed C3: 47uF 50V, Capacitor_SMD:CP_Elec_6.3x7.7, symbol Device:C_Small
- added C3: 47uF 50V, Capacitor_SMD:CP_Elec_6.3x7.7, symbol Device:C_Polarized
- C2: value 100nF -> 100nF 50V; BOM Comments Tu 104 100nF 0805 50V - Mua tai CXT: linhkien.cxtvn.com/197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 -> (none); LCSC Part C49678 -> (none); Link to Buy (none) -> https://linhkien.cxtvn.com/1976-tu-khong-phan-cuc-0805.html; MPN CC0805KRX7R9BB104 -> (none); Manufacturer Yageo -> (none)
- D2: BOM Comments Mua tai LKCL: linhkienchatluong.vn/urldiode-chinh-luu/diode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 -> (none); LCSC Part C84410 -> (none); Link to Buy (none) -> https://linhkien.cxtvn.com/7017-1n4148w-7-f-diode-gen-purp-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; MPN 1N4148W -> (none); Manufacturer JCET -> (none)
- D7: footprint Diode_THT:D_DO-41_SOD81_P10.16mm_Horizontal -> Diode_SMD:Nexperia_CFP3_SOD-123W; BOM Comments FR107 Diode xung 1A 1000V DO-41 - Mua tai CXT: linhkien.cxt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 -> (none); LCSC Part C35253 -> (none); Link to Buy (none) -> https://linhkien.cxtvn.com/9278-rs1m-fr107-f7-diode-xung-1a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; MPN FR107 -> (none)
- Q8: BOM Comments Mua tai LKCL: linhkienchatluong.vn/transistor/bc817-40-6c-6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 -> (none); LCSC Part C5205285 -> (none); Link to Buy (none) -> https://linhkien.cxtvn.com/5979-bc817-40-transistor-npn-45v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; MPN BC817-40 -> (none); Manufacturer NXP -> (none)
- R83: BOM Comments Dien tro dan 0805 1% - Mua tai CXT: linhkien.cxtvn.com/6337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 -> (none); LCSC Part C17710 -> (none); Link to Buy (none) -> Dien tro dan 0805 1% - Mua tai CXT: linhkien.cxtvn.com/6337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; MPN 0805W8F4700T5E -> (none); Manufacturer UniOhm -> (none)
- R84: BOM Comments Dien tro dan 0805 1% - Mua tai CXT: linhkien.cxtvn.com/6337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 -> (none); LCSC Part C26010 -> (none); Link to Buy (none) -> https://linhkien.cxtvn.com/4177-dien-tro-0805-1-thong-so-tu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; MPN 0805W8F3301T5E -> (none); Manufacturer UniOhm -> (none)
- R85: BOM Comments Dien tro dan 0805 1% - Mua tai CXT: linhkien.cxtvn.com/6337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 -> (none); LCSC Part C17414 -> (none); Link to Buy (none) -> Dien tro dan 0805 1% - Mua tai CXT: linhkien.cxtvn.com/6337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; MPN 0805W8F1002T5E -> (none); Manufacturer UniOhm -> (none)
- U13: BOM Comments Thay LTV-357T bang LTV-354T (pin-compatible). Mua tai CXT: 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 -> (none); LCSC Part C119089 -> (none); Link to Buy (none) -> Thay LTV-357T bang LTV-354T (pin-compatible). Mua tai CXT: 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; MPN LTV-354T -> (none); Manufacturer Lite-On -> (none)
- U8: footprint easyeda2kicad:RELAY-TH_HF116F-80-XX-1HTF -> HF116F-80-12-24-1HTF:RELAY-TH_HF116F-80-XX-1HTF; BOM Comments Relay HV 80A - khong ban le tai VN. Dat tu LCSC: C5322130 (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 -> (none); LCSC Part C5322130 -> (none); Link to Buy (none) -> Relay HV 80A - khong ban le tai VN. Dat tu LCSC: C5322130 (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; MPN HF116F-80/24-1HTF -> (none); Manufacturer HF(宏发) -> (none)
Connections:
- net +24V: now also C3.1
- net GND: now also C2.2, C3.2
- net VBAT_PROTECTED_P: no longer C2.2
Other:
- moved on the sheet: C2, R83

Commit message: feat: update buy link, footprint
Parts:
- R85: Link to Buy Dien tro dan 0805 1% - Mua tai CXT: linhkien.cxtvn.com/6337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 -> https://linhkien.cxtvn.com/8792-dien-tro-10k-0805-01-10c.ht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
Changed lines of the file:
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@@
 			)
 		)
-		(property "Link to Buy" "Dien tro dan 0805 1% - Mua tai CXT: linhkien.cxtvn.com/6337-dien-tro-0805-1-thong-so-tu-1k-den-91k.html (chon 10k)"
+		(property "Link to Buy" "https://linhkien.cxtvn.com/8792-dien-tro-10k-0805-01-10c.html"
 			(at 0 0 0)
 			(hide yes)

Commit message: feat: update schematic with new components for communication interfaces and export BOM list
Parts:
- removed Q8: BC817-40, Package_TO_SOT_SMD:SOT-23, symbol Transistor_BJT:BC817
- added D17: BZT52C12, Diode_SMD:D_SOD-123, symbol Diode:1N914
- added Q8: SI2308BDS, Package_TO_SOT_SMD:SOT-23, symbol Transistor_FET:2N7002K
- C2: value 100nF 50V -> 100nF
- C3: value 47uF 50V -> 47uF
- D7: value FR107 -> RS1M; footprint Diode_SMD:Nexperia_CFP3_SOD-123W -> Diode_SMD:D_SOD-123
- R83: value 470R -> 220R; Link to Buy Dien tro dan 0805 1% - Mua tai CXT: linhkien.cxtvn.com/6337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 -> https://linhkien.cxtvn.com/2345-dien-tro-470r-0805-1-100c.h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
- R84: value 3.3k -> 3.3kR
- R85: value 10k -> 10kR; Link to Buy https://linhkien.cxtvn.com/8792-dien-tro-10k-0805-01-10c.ht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 -> https://linhkien.cxtvn.com/9909-dien-tro-0805-05-18w-10-chi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
- U13: value LTV-354T -> LTV-357T; LCSC Part (none) -> C119091; Link to Buy Thay LTV-357T bang LTV-354T (pin-compatible). Mua tai CXT: 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 -> https://linhkienchatluong.vn/urlltv/ltv357-ltv357t-sop-4-ch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; MPN (none) -> LTV-357T; Manufacturer (none) -> Lite-On
Connections:
- net GND: now also U13.3, D17.2 (A), Q8.3 (D); no longer U13.2
- net MAIN_RELAY_COIL_N: now also Q8.2 (S)
- net at R83.2: now also U13.4; no longer U13.1
- net at R85.2: now also U13.2, D17.1 (K), Q8.1 (G); no longer U13.3
- net at R84.1: now also U13.1; no longer U13.4
Other:
- moved on the sheet: R83, R85

Commit message: Refactor code structure for improved readability and maintainability
Connections:
- net GND: now also Q8.2 (S); no longer Q8.3 (D)
- net MAIN_RELAY_COIL_N: now also Q8.3 (D); no longer Q8.2 (S)
Other:
- moved on the sheet: Q8
Changed lines of the file:
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@@
 	(symbol
 		(lib_id "Transistor_FET:2N7002K")
-		(at 185.42 78.74 180)
+		(at 185.42 78.74 0)
+		(mirror y)
 		(unit 1)
 		(body_style 1)
@@
 		(in_pos_files yes)
 		(dnp no)
-		(fields_autoplaced yes)
 		(property "Reference" "Q8"
-			(at 179.07 77.4699 0)
+			(at 179.07 80.0101 0)
 			(show_name no)
 			(do_not_autoplace no)
@@
 		)
 		(property "Value" "SI2308BDS"
-			(at 179.07 80.0099 0)
+			(at 179.07 77.4701 0)
 			(show_name no)
 			(do_not_autoplace no)
@@
 		)
 		(property "Footprint" "Package_TO_SOT_SMD:SOT-23"
-			(at 180.34 76.835 0)
+			(at 180.34 80.645 0)
 			(hide yes)
 			(show_name no)
@@
 		)
 		(property "Datasheet" "https://www.vishay.com/docs/69958/si2308bds.pdf"
-			(at 180.34 74.93 0)
+			(at 180.34 82.55 0)
 			(hide yes)
 			(show_name no)
