File: Hardware/One_Board_Design/MCU_Control.kicad_sch (KiCad schematic)
At the start: 19 parts, among them J1 USB2.0_16P, Q3 BC817, Q4 BC817, SW1 ENABLE, U15 CH340C, U4 ESP32-WROOM-32E, U5 USBLC6-2SC6

Commit message: refactor(hardware): move KiCad project into One_Board_Design/
Relocate the single-board KiCad project (root schematic, five hierarchical sheets, PCB, project file, and library tables) into Hardware/One_Board_Design/ so the shared symbols, footprints, and 3D models stay in Hardware/libraries/.

Update library tables and 3D model references to use \/../libraries/... so the moved project resolves the shared library location correctly. Replace SparkFun symbol references with the equivalent KiCad standard symbols. Add One_Board_Design README documenting the shared-library layout.

Ultraworked with [Sisyphus](https://github.com/code-yeongyu/oh-my-openagent)

Co-authored-by: Sisyphus <clio-agent@sisyphuslabs.ai>
Parts:
- C15, C24, C43: symbol SparkFun-Capacitor:C -> Device:C
Changed lines of the file:
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@@
 	)
 	(symbol
-		(lib_id "SparkFun-PowerSymbol:3.3V")
+		(lib_id "power:+3.3V")
 		(at 172.72 41.91 0)
 		(unit 1)
@@
 	)
 	(symbol
-		(lib_id "SparkFun-PowerSymbol:3.3V")
+		(lib_id "power:+3.3V")
 		(at 81.28 72.39 0)
 		(unit 1)
@@
 	)
 	(symbol
-		(lib_id "SparkFun-Capacitor:C")
+		(lib_id "Device:C")
 		(at 35.56 124.46 0)
 		(unit 1)
@@
 	)
 	(symbol
-		(lib_id "SparkFun-Capacitor:C")
+		(lib_id "Device:C")
 		(at 127.254 57.15 0)
 		(unit 1)
@@
 	)
 	(symbol
-		(lib_id "SparkFun-Capacitor:C")
+		(lib_id "Device:C")
 		(at 101.6 82.55 0)
 		(mirror y)
@@
 	)
 	(symbol
-		(lib_id "SparkFun-PowerSymbol:3.3V")
+		(lib_id "power:+3.3V")
 		(at 93.98 41.91 0)
 		(unit 1)
@@
 	)
 	(symbol
-		(lib_id "SparkFun-PowerSymbol:3.3V")
+		(lib_id "power:+3.3V")
 		(at 60.96 110.49 0)
 		(unit 1)
