File: Hardware/One_Board_Design/Output_Protection_And_Sensing.kicad_sch (KiCad schematic)
At the start: 15 parts, among them U2 INA240A1PW

Commit message: refactor(hardware): move KiCad project into One_Board_Design/
Relocate the single-board KiCad project (root schematic, five hierarchical sheets, PCB, project file, and library tables) into Hardware/One_Board_Design/ so the shared symbols, footprints, and 3D models stay in Hardware/libraries/.

Update library tables and 3D model references to use \/../libraries/... so the moved project resolves the shared library location correctly. Replace SparkFun symbol references with the equivalent KiCad standard symbols. Add One_Board_Design README documenting the shared-library layout.

Ultraworked with [Sisyphus](https://github.com/code-yeongyu/oh-my-openagent)

Co-authored-by: Sisyphus <clio-agent@sisyphuslabs.ai>
Parts:
- R41, R49, R50: footprint CSS2H_2512R_1L00F:RES_1L00x_BRN -> RobotChargeController:RES_1L00x_BRN
Changed lines of the file:
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@@
 			)
 		)
-		(property "Footprint" "CSS2H_2512R_1L00F:RES_1L00x_BRN"
+		(property "Footprint" "RobotChargeController:RES_1L00x_BRN"
 			(at 133.35 68.58 0)
 			(hide yes)
@@
 			)
 		)
-		(property "Footprint" "CSS2H_2512R_1L00F:RES_1L00x_BRN"
+		(property "Footprint" "RobotChargeController:RES_1L00x_BRN"
 			(at 133.35 59.69 0)
 			(hide yes)
@@
 			)
 		)
-		(property "Footprint" "CSS2H_2512R_1L00F:RES_1L00x_BRN"
+		(property "Footprint" "RobotChargeController:RES_1L00x_BRN"
 			(at 133.35 52.07 0)
 			(hide yes)
