File: hardware/One_Board_Design/robot-hv-charge-controller.kicad_pcb (KiCad board)
At the start: 2 copper layers, 100 x 100 mm, 132 parts, among them J1 USB2.0_16P, J2 UART_CONN, J3 XT30PW-M, J4 Conn_01x02, J5 XT60PW-M, J6 Conn_01x02, J7 XT60PW-M, J8 Conn_01x03, J9 Conn_01x02, Q2 2SD882, Q3 BC817, Q4 BC817, Q5 2SD882, Q6 2SD882, Q7 MJD41CT4G, SW1 ENABLE, U1 TCAN3414DR, U10 LTV-356T, U11 LTV-356T, U12 LTV-356T, U13 LTV-356T, U14 LTV-356T, U15 CH340C, U2 INA240A1PW, U3 MAX3485, U4 ESP32-WROOM-32E, U5 USBLC6-2SC6, U6 LTV-356T, U7 TLV1117-33, U8 HF116F-80/24-1HTF, U9 LV14340DDAR

Commit message: upđate: Some minor change in PCB
Routing:
- net GND: track 161.8 -> 160.5 mm
Changed lines of the file:
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@@
 		(tags "resistor")
 		(property "Reference" "R47"
-			(at 2.75 -0.06 90)
+			(at 3.28 -0.05 90)
 			(layer "F.SilkS")
 			(effects
@@
 		(tags "SOIC SO")
 		(property "Reference" "U3"
-			(at 2.77 4.12 0)
+			(at 2.86 3.31 0)
 			(layer "F.SilkS")
 			(effects
@@
 		(tags "LV14340DDAR ")
 		(property "Reference" "U9"
-			(at 0.82 3.44 0)
+			(at 1.05 3.61 0)
 			(unlocked yes)
 			(layer "F.SilkS")
@@
 		(tags "LED")
 		(property "Reference" "D14"
-			(at 0 -1.37 0)
+			(at 0 -1.65 0)
 			(layer "F.SilkS")
 			(effects
@@
 		(tags "capacitor")
 		(property "Reference" "C23"
-			(at -2.7025 0 0)
+			(at -3.63 0 0)
 			(layer "F.SilkS")
 			(effects
@@
 		(tags "resistor")
 		(property "Reference" "R4"
-			(at -1.98 -0.005 0)
+			(at -2.17 0.03 0)
 			(layer "F.SilkS")
 			(effects
@@
 		(tags "capacitor")
 		(property "Reference" "C45"
-			(at 0 -1.43 90)
+			(at 0 -2.52375 180)
 			(layer "F.SilkS")
 			(effects
@@
 		(tags "resistor")
 		(property "Reference" "R58"
-			(at -0.02 1.36 90)
+			(at -0.0375 1.39625 90)
 			(layer "F.SilkS")
 			(effects
 				(font
-					(size 1 1)
+					(size 0.8 0.8)
 					(thickness 0.15)
 				)
@@
 		(tags "resistor")
 		(property "Reference" "R28"
-			(at -2.705 0.04 90)
+			(at -3.235 0.03 90)
 			(layer "F.SilkS")
 			(effects
@@
 		(tags "capacitor")
 		(property "Reference" "C30"
-			(at 2.29 -0.04 180)
+			(at -0.0125 -2.2275 180)
 			(layer "F.SilkS")
 			(effects
@@
 		(tags "capacitor")
 		(property "Reference" "C46"
-			(at 0 -1.43 90)
+			(at 0.0575 -2.37625 180)
 			(layer "F.SilkS")
 			(effects
@@
 		(tags "fuse")
 		(property "Reference" "F2"
-			(at 3.04 0.01 0)
+			(at 3.8 0.11 0)
 			(layer "F.SilkS")
 			(effects
@@
 		(tags "SOIC SO 16-pin-NSOP R-16 R-16-S D0016A M2B SO16 SOT109-1 751B SOIC_N narrow")
 		(property "Reference" "U15"
-			(at -4.21 -5.65 0)
+			(at -3.95 -5.9575 0)
 			(layer "F.SilkS")
 			(effects
@@
 		(tags "resistor")
 		(property "Reference" "R74"
-			(at -2.67 0.01 180)
+			(at 0.02 1.625 180)
 			(layer "F.SilkS")
 			(effects
@@
 		(tags "capacitor")
 		(property "Reference" "C28"
-			(at -2.36 -0.0175 180)
+			(at 0 2.1825 180)
 			(layer "F.SilkS")
 			(effects
@@
 		(tags "resistor")
 		(property "Reference" "R5"
-			(at 2.23 0.01 0)
+			(at 2.42 -0.01 0)
 			(layer "F.SilkS")
 			(effects
@@
 		(tags "resistor")
 		(property "Reference" "R8"
-			(at -2.23 0.02 0)
+			(at -2.42 0.02 0)
 			(layer "F.SilkS")
 			(effects
@@
 		(tags "capacitor")
 		(property "Reference" "C31"
-			(at -2.735 0.04 90)
+			(at -3.265 0.03 90)
 			(layer "F.SilkS")
 			(effects
@@
 		(tags "SOT TO_SOT_SMD")
 		(property "Reference" "D10"
-			(at -1.34 -2.86 0)
+			(at -1.2225 -3.87 0)
 			(layer "F.SilkS")
 			(effects
@@
 		(tags "resistor")
 		(property "Reference" "R77"
-			(at -2.66 0.02 0)
+			(at -0.01 1.54 0)
 			(layer "F.SilkS")
 			(effects
@@
 		(tags "capacitor")
 		(property "Reference" "C26"
-			(at 2.68 0 90)
+			(at 3.21 0.01 90)
 			(layer "F.SilkS")
 			(effects
@@
 		(tags "resistor")
 		(property "Reference" "R10"
-			(at 0 1.33 0)
+			(at 0 1.54 0)
 			(layer "F.SilkS")
 			(effects
@@
 		(tags "resistor")
 		(property "Reference" "R80"
-			(at -2.875 0 0)
+			(at 0.02 1.5925 0)
 			(layer "F.SilkS")
 			(effects
@@
 		)
 		(embedded_fonts no)
-		(model "kicad-embed://R_0603_1608Metric.step"
+		(model "${KIPRJMOD}/../libraries/3d-models/R_0603_1608Metric.step"
 			(offset
 				(xyz 0 0 0)
@@
 		(tags "SOIC SO")
 		(property "Reference" "U1"
-			(at -4.45 2.0925 0)
+			(at 0.01375 3.515 0)
 			(layer "F.SilkS")
 			(effects
@@
 		(tags "capacitor")
 		(property "Reference" "C42"
-			(at -3.0125 -0.02 0)
+			(at -3.51 -0.01 0)
 			(layer "F.SilkS")
 			(effects
@@
 		(tags "capacitor")
 		(property "Reference" "C4"
-			(at 2.01 0 90)
+			(at 2.1 -0.18 90)
 			(layer "F.SilkS")
 			(effects
@@
 	)
 	(segment
-		(start 164.16625 49.3625)
-		(end 164.16625 48.1075)
-		(width 0.25)
-		(layer "F.Cu")
-		(net "GND")
-	)
-	(segment
 		(start 166.08 128.39)
 		(end 166.06 128.41)
@@
 	)
 	(segment
-		(start 193.445 62.4625)
-		(end 194.8575 63.875)
+		(start 193.87 72.89)
+		(end 188.4975 72.89)
 		(width 0.35)
 		(layer "B.Cu")
-		(net "DO1_SINK")
+		(net "DO3_SINK")
 	)
 	(segment
-		(start 194.8575 63.2575)
-		(end 194.8575 63.875)
-		(width 0.4)
+		(start 194.06 72.71)
+		(end 194.05 72.71)
+		(width 0.25)
 		(layer "B.Cu")
-		(net "DO1_SINK")
+		(net "DO3_SINK")
 	)
 	(segment
-		(start 188.4875 62.4625)
-		(end 193.445 62.4625)
+		(start 188.085 72.9)
+		(end 188.4875 72.9)
 		(width 0.35)
 		(layer "B.Cu")
-		(net "DO1_SINK")
+		(net "DO3_SINK")
 	)
 	(segment
-		(start 188.4875 62.4625)
-		(end 188.1175 62.4625)
+		(start 188.4975 72.89)
+		(end 188.4875 72.9)
+		(width 0.25)
+		(layer "B.Cu")
+		(net "DO3_SINK")
+	)
+	(segment
+		(start 194.06 72.71)
+		(end 194.8575 71.9125)
 		(width 0.35)
 		(layer "B.Cu")
-		(net "DO1_SINK")
+		(net "DO3_SINK")
 	)
 	(segment
-		(start 188.1175 62.4625)
-		(end 186.77 61.115)
+		(start 194.8575 71.9125)
+		(end 194.8575 71.495)
 		(width 0.35)
 		(layer "B.Cu")
-		(net "DO1_SINK")
+		(net "DO3_SINK")
+	)
+	(segment
+		(start 194.05 72.71)
+		(end 193.87 72.89)
+		(width 0.35)
+		(layer "B.Cu")
+		(net "DO3_SINK")
+	)
+	(segment
+		(start 186.7425 71.5575)
+		(end 188.085 72.9)
+		(width 0.35)
+		(layer "B.Cu")
+		(net "DO3_SINK")
 	)
 	(segment
@@
 	)
 	(segment
-		(start 193.87 72.89)
-		(end 188.4975 72.89)
-		(width 0.35)
-		(layer "B.Cu")
-		(net "DO3_SINK")
-	)
-	(segment
-		(start 194.06 72.71)
-		(end 194.05 72.71)
-		(width 0.25)
-		(layer "B.Cu")
-		(net "DO3_SINK")
-	)
-	(segment
-		(start 188.085 72.9)
-		(end 188.4875 72.9)
+		(start 193.445 62.4625)
+		(end 194.8575 63.875)
 		(width 0.35)
 		(layer "B.Cu")
-		(net "DO3_SINK")
-	)
-	(segment
-		(start 188.4975 72.89)
-		(end 188.4875 72.9)
-		(width 0.25)
-		(layer "B.Cu")
-		(net "DO3_SINK")
+		(net "DO1_SINK")
 	)
 	(segment
-		(start 194.06 72.71)
-		(end 194.8575 71.9125)
-		(width 0.35)
+		(start 194.8575 63.2575)
+		(end 194.8575 63.875)
+		(width 0.4)
 		(layer "B.Cu")
-		(net "DO3_SINK")
+		(net "DO1_SINK")
 	)
 	(segment
-		(start 194.8575 71.9125)
-		(end 194.8575 71.495)
+		(start 188.4875 62.4625)
+		(end 193.445 62.4625)
 		(width 0.35)
 		(layer "B.Cu")
-		(net "DO3_SINK")
+		(net "DO1_SINK")
 	)
 	(segment
-		(start 194.05 72.71)
-		(end 193.87 72.89)
+		(start 188.4875 62.4625)
+		(end 188.1175 62.4625)
 		(width 0.35)
 		(layer "B.Cu")
-		(net "DO3_SINK")
+		(net "DO1_SINK")
 	)
 	(segment
-		(start 186.7425 71.5575)
-		(end 188.085 72.9)
+		(start 188.1175 62.4625)
+		(end 186.77 61.115)
 		(width 0.35)
 		(layer "B.Cu")
-		(net "DO3_SINK")
+		(net "DO1_SINK")
 	)
 	(segment
