File: hardware/Split_Board_Design/Relay_Board/Output_Sensing.kicad_sch (KiCad schematic)
At the start: 20 parts, among them U2 INA240A2PW

Commit message: feat(layout): Update layout
Parts:
- removed R13, R14, R15, R16, R17, R18: 1R, Resistor_SMD:R_0603_1608Metric, symbol Device:R_Small
- C30: value 100nF -> 100nF-50V
Connections:
- net VBAT_RELAY_OUT_P: now also R1.3 (V_A), R2.3 (V_A), R3.3 (V_A), U2.2 (+)
- net VBAT_SEN_OUT_P: now also R1.4 (V_B), R2.4 (V_B), R3.4 (V_B), U2.3 (-)
Other:
- moved on the sheet: C30

Commit message: Some minor updates
Parts:
- C31: value 10nF-50V -> 100nF-50V; Link to Buy https://linhkien.cxtvn.com/6736-0603b104k500nt-tu-100nf-50v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 -> https://linhkien.cxtvn.com/1981-tu-0603-khong-phan-cuc.html
- R42: value 10kR -> 1kR; Link to Buy https://linhkien.cxtvn.com/1422-dien-tro-10k-0603-1-100c.ht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 -> https://linhkien.cxtvn.com/1424-dien-tro-1k-0603-1-100c.html
Other:
- moved on the sheet: R1, R2

Commit message: feat(layout): update relay board layout
Parts:
- removed R1, R2, R3: 2mR, RobotChargeController:R_Shunt_FOJAN_2512L_4Terminal_Kelvin_C, symbol RobotChargeController:FPM253WFR002TML_4Terminal_Kelvin
- removed U2: INA240A2PW, Package_SO:TSSOP-8_4.4x3mm_P0.65mm, symbol Amplifier_Current:INA240A1PW
- added R48, R49, R50: 2mR, RobotChargeController:R_Shunt_FOJAN_2512L_4Terminal_Kelvin_C, symbol Device:R_Small
- added U1: INA240A2D, Package_SO:SOIC-8_3.9x4.9mm_P1.27mm, symbol Amplifier_Current:INA240A2D
Connections:
- net +3V3: now also U1.6 (V+), U1.7 (REF1)
- net GND: now also U1.2 (GND), U1.3 (REF2), U1.4 (GND)
- net VBAT_RELAY_OUT_P: now also R48.1, R49.1, R50.1, U1.8 (+)
- net VBAT_SEN_OUT_P: now also R48.2, R49.2, R50.2, U1.1 (-)
- net at R47.2: now also U1.5
Other:
- moved on the sheet: C29, C30, C31, R42, R43, R44, R45, R46, R47, R54
