File: hardware/Split_Board_Design/Relay_Board/Relay_control.kicad_sch (KiCad schematic)
At the start: 9 parts, among them Q7 MJD41CT4G, U13 LTV-356T, U8 HF116F-80/24-1HTF

Commit message: feat(layout): Finish demo layout of relay board
Parts:
- C2: Link to Buy https://linhkien.cxtvn.com/1976-tu-khong-phan-cuc-0805.html -> https://linhkien.cxtvn.com/6736-0603b104k500nt-tu-100nf-50v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
- C3: value 100uF-50V -> 680uf-35v; footprint Capacitor_SMD:CP_Elec_8x10.5 -> RobotChargeController:CP_Elec_12.5x13.5_Generic_H13; Link to Buy https://linhkien.cxtvn.com/3033-tu-nhom-100uf-50v-8x105-5c.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 -> https://linhkien1993.com/tu-nhom-smd-680uf-35v-12-5x13-5mm
- D7: Link to Buy https://banlinhkiendientu.vn/us1m-uf4007/ -> https://linhkien.cxtvn.com/9736-her107-us1m-diode-1a-1000v-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
- Q7: Link to Buy (none) -> https://cungcaplinhkien.vn/transistor-dan-tip41c-sm-to252-s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
- R83: Link to Buy https://linhkien.cxtvn.com/1958-dien-tro-0805-5-thong-so-10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 -> https://linhkien.cxtvn.com/9913-dien-tro-1k-0805-05-18w-20c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
- R84: Link to Buy https://linhkien.cxtvn.com/4177-dien-tro-0805-1-thong-so-tu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 -> https://linhkien.cxtvn.com/4177-dien-tro-33k-0805-1-100c.ht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
- R85: Link to Buy https://linhkien.cxtvn.com/9909-dien-tro-0805-05-18w-10-chi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 -> https://linhkien.cxtvn.com/8792-dien-tro-10k-0805-01-10c.ht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

Commit message: feat(layout): update relay board layout
Parts:
- removed C2: 100nF-50V, Capacitor_SMD:C_0805_2012Metric, symbol Device:C_Small
Other:
- moved on the sheet: C3
