File: hardware/Split_Board_Design/Control_Board/control-board.kicad_pcb (KiCad board)
At the start: 2 copper layers, 100 x 60 mm, 111 parts, among them J1 USB2.0_16P, J10 Conn_01x03, J2 UART_CONN, J3 XT30PW-M, J5 Conn_01x06, J7 Conn_01x03, J8 Conn_01x03, J9 Conn_01x02, Q2 2SD882, Q3 BC817, Q4 BC817, Q5 2SD882, Q6 2SD882, SW1 ENABLE, U1 TCAN3414DR, U10 LTV-356T, U11 LTV-356T, U12 LTV-356T, U14 LTV-356T, U15 CH340C, U3 MAX3485, U4 ESP32-WROOM-32E, U5 USBLC6-2SC6, U6 LTV-356T, U7 TLV1117-33, U8 LV14340DDAR

Commit message: layout: update layout
Parts:
- removed C28: 10uF-50V, Capacitor_SMD:C_0603_1608Metric
- removed J3: XT30PW-M, RobotChargeController:AMASS_XT30PW-M
- added C22: 10uF-50V, Capacitor_SMD:C_0603_1608Metric, F.Cu at (173.8, 85.2)
- added G***: LOGO, RobotChargeController:MSVN_LOGO, F.Cu at (162.7, 93.0)
- added J11: Conn_01x02, Connector_Phoenix_MC:PhoenixContact_MC_1,5_2-G-3.81_1x02_P3.81mm_Horizontal, F.Cu at (107.1, 87.5)
- C1: value 680uF-35V -> 100uF-50V; footprint RobotChargeController:CP_Elec_12.5x13.5_Generic_H13 -> Capacitor_SMD:CP_Elec_8x10.5
- D19, D20, D21, D23: footprint Diode_SMD:D_SOD-323 -> Diode_SMD:D_SOD-523
- D4: value SMAJ36CA -> SMAJ24A
- J2: footprint Connector_JST:JST_XH_S4B-XH-A-1_1x04_P2.50mm_Horizontal -> RobotChargeController:JST_XH_S4B-XH-A-1_1x04_P2.50mm_Horizontal
- J5: footprint Connector_JST:JST_XH_S6B-XH-A_1x06_P2.50mm_Horizontal -> RobotChargeController:JST_XH_S6B-XH-A_1x06_P2.50mm_Horizontal
- Q3, Q4: footprint Package_TO_SOT_SMD:SOT-23 -> Package_TO_SOT_SMD:SOT-23-3
- R10: value 49.9R -> 49.9kR
- moved D1 10.5 mm to (192.6, 112.3)
- moved F3 10.1 mm to (111.7, 92.7), turned to -90 degrees
- moved D5 10.0 mm to (192.6, 102.7)
- moved D6 9.98 mm to (192.6, 96.8)
- moved C23 7.35 mm to (142.5, 95.4), turned to 180 degrees
- moved U7 4.51 mm to (140.7, 99.7), turned to 0 degrees
- moved C42 4.12 mm to (142.5, 93.9), turned to 180 degrees
- moved R33 3.71 mm to (172.5, 78.8), turned to 90 degrees
- moved R34 3.53 mm to (172.5, 82.3)
- moved D4 2.85 mm to (113.7, 97.1)
- moved D3 2.77 mm to (113.7, 100.8)
- moved C46 2.67 mm to (127.1, 72.2)
- moved D12 2.61 mm to (129.6, 72.6)
- moved R55 2.61 mm to (125.3, 82.1)
- moved U1 2.61 mm to (129.7, 81.1)
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Connections:
- D3 pad 1: Net-(D3-K) -> +24V
- D3 pad 2: /Auxiliary_Power_Supply/VAUX_IN_P -> Net-(D3-A)
- D4 pad 1: /Auxiliary_Power_Supply/VAUX_IN_P -> Net-(D3-A)
- F3 pad 1: Net-(D3-K) -> /Auxiliary_Power_Supply/VAUX_IN_P
- F3 pad 2: +24V -> Net-(D3-A)
- J5 pad 6: +24V -> GND
- U15 pad 16: V_USB -> +3V3
Routing:
- net V_USB: track 27.4 -> 10.2 mm
- net +5V: track 176.6 -> 164.5 mm
- net GND: track 36.1 -> 26.3 mm, vias 894 -> 545
- net +3V3: track 171.3 -> 180.3 mm, vias 7 -> 9
- net /Auxiliary_Power_Supply/VAUX_IN_P: track 13.4 -> 4.58 mm
- net Net-(D3-A): track 0.00 -> 6.69 mm
- net Net-(Q4-B): track 8.18 -> 1.90 mm
- net /MCU_Control/USB_UART_DTR: track 9.55 -> 4.89 mm, vias 2 -> 0
- net +24V: track 141.3 -> 136.9 mm
- net Net-(D3-K): track 3.81 -> 0.00 mm
- net /Communication_Interfaces/CAN_RX: track 18.0 -> 20.7 mm
- net /Communication_Interfaces/CAN_TX: track 20.5 -> 23.0 mm
- net Net-(Q3-B): track 4.95 -> 2.78 mm, vias 2 -> 0
- net DO2_SINK: track 11.4 -> 13.2 mm
- net /Communication_Interfaces/SW2_SENSE_N: track 32.6 -> 31.3 mm
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Other:
- board text added: "DI1 DI2"
- board text added: "DO1 D02 D03"
- board text added: "ROBOT CHARGE CONTROLLER V1.0"
- board text added: "Vo Io 3V3 GND CTR GND"
- board text added: "{ "ViaStitching": "0.3.0", "stitch_zone_0": { "HSpacing": "1.5", "VSpacing": "1.5", "HOffset": "0", "VOffset": "0", "Clearance": "0.5", "Randomize": false, "Stagger": false, "OnlyFilledCopper": true } }"
- board text added: "{ "ViaStitching": "0.3.0", "stitch_zone_0": { "HSpacing": "3", "VSpacing": "3", "HOffset": "0", "VOffset": "0", "Clearance": "0.5", "Randomize": false, "Stagger": false, "OnlyFilledCopper": true } }"
- board text added: "{ "ViaStitching": "0.3.0", "stitch_zone_0": { "HSpacing": "3", "VSpacing": "3", "HOffset": "0", "VOffset": "0", "Clearance": "0.5", "Randomize": true, "Stagger": false, "OnlyFilledCopper": true } }"
- board text added: "{ "ViaStitching": "0.3.0", "stitch_zone_0": { "HSpacing": "3", "VSpacing": "3", "HOffset": "0", "VOffset": "0", "Clearance": "0.5", "Randomize": true, "Stagger": true, "OnlyFilledCopper": true } }"
- board text removed: "24V CTR GND 3V3 Vo Io"
- board text removed: "G"
- board text removed: "R"
- board text removed: "SW1"
- board text removed: "SW2"
- board text removed: "Y"
